File: oshpark-4layer/oshpark-4layer.kicad_sch (KiCad schematic)
At the start: 0 parts

Commit message: Use project variables for the title blocks.
Also change the paper sizes from USLetter and USLedger to A and B.
Other:
- company: (none) -> ${COMPANY}
- title: OSH Park 4-layer template -> ${TITLE}
Changed lines of the file:
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@@
 (kicad_sch (version 20211123) (generator eeschema)
-  (paper "USLedger")
+  (paper "B")
   (title_block
-    (title "OSH Park 4-layer template")
-    (date "2022-05-04")
-    (rev "A")
+    (title "${TITLE}")
+    (date "${DATE}")
+    (rev "${REVISION}")
+    (company "${COMPANY}")
   )
   (sheet_instances
